File: Panthera.kicad_pcb (KiCad board)
At the start: 2 copper layers, 69.9 x 42.2 mm, 12 parts, among them IC1 TEENSY_4.1, SW1 SW_SPDT

Commit message: Updated PCB
Parts:
- renumbered MPU1 to BME1, ACC1 to MPU1
Changed lines of the file:
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@@
 	)
 	(net 0 "")
-	(net 1 "unconnected-(ACC1-XDA-Pad5)")
-	(net 2 "unconnected-(ACC1-AD0-Pad7)")
+	(net 1 "unconnected-(BME1-SDO-Pad6)")
+	(net 2 "Net-(BME1-SCL)")
 	(net 3 "+3.3V")
-	(net 4 "unconnected-(ACC1-INT-Pad8)")
-	(net 5 "Net-(ACC1-SCL)")
+	(net 4 "Net-(BME1-SDA)")
+	(net 5 "unconnected-(BME1-CSB-Pad5)")
 	(net 6 "GND")
-	(net 7 "Net-(ACC1-SDA)")
-	(net 8 "unconnected-(ACC1-XCL-Pad6)")
-	(net 9 "Net-(IC1-A3)")
+	(net 7 "Net-(IC1-A4)")
+	(net 8 "Net-(IC1-A5)")
+	(net 9 "unconnected-(MPU1-XDA-Pad5)")
 	(net 10 "unconnected-(IC1-OUT1C-Pad9)")
 	(net 11 "unconnected-(IC1-A8-Pad22)")
@@
 	(net 20 "/MOSI")
 	(net 21 "unconnected-(IC1-VBAT-Pad43)")
-	(net 22 "Net-(IC1-A2)")
+	(net 22 "unconnected-(MPU1-AD0-Pad7)")
 	(net 23 "unconnected-(IC1-MCLK2-Pad33)")
 	(net 24 "unconnected-(IC1-IN2-Pad5)")
@@
 	(net 58 "unconnected-(Lora1-DIO2-Pad7)")
 	(net 59 "unconnected-(Lora1-DIO5-Pad11)")
-	(net 60 "unconnected-(MPU1-SDO-Pad6)")
-	(net 61 "unconnected-(MPU1-CSB-Pad5)")
+	(net 60 "unconnected-(MPU1-INT-Pad8)")
+	(net 61 "unconnected-(MPU1-XCL-Pad6)")
 	(net 62 "/RESET")
 	(net 63 "unconnected-(IC1-OUT1D-Pad6)")
@@
 		(layer "F.Cu")
 		(at 144.78 78.994 -90)
-		(property "Reference" "ACC1"
+		(property "Reference" "MPU1"
 			(at -3.494 8.28 0)
 			(unlocked yes)
@@
 			)
 			(fill none)
-			(layer "Dwgs.User")
+			(layer "F.SilkS")
 		)
 		(fp_line
@@
 			(layers "*.Cu" "*.Mask")
 			(remove_unused_layers no)
-			(net 5 "Net-(ACC1-SCL)")
+			(net 8 "Net-(IC1-A5)")
 			(pinfunction "SCL")
 			(pintype "bidirectional")
@@
 			(layers "*.Cu" "*.Mask")
 			(remove_unused_layers no)
-			(net 7 "Net-(ACC1-SDA)")
+			(net 7 "Net-(IC1-A4)")
 			(pinfunction "SDA")
 			(pintype "bidirectional")
@@
 			(layers "*.Cu" "*.Mask")
 			(remove_unused_layers no)
-			(net 1 "unconnected-(ACC1-XDA-Pad5)")
+			(net 9 "unconnected-(MPU1-XDA-Pad5)")
 			(pinfunction "XDA")
 			(pintype "bidirectional+no_connect")
@@
 			(layers "*.Cu" "*.Mask")
 			(remove_unused_layers no)
-			(net 8 "unconnected-(ACC1-XCL-Pad6)")
+			(net 61 "unconnected-(MPU1-XCL-Pad6)")
 			(pinfunction "XCL")
 			(pintype "bidirectional+no_connect")
@@
 			(layers "*.Cu" "*.Mask")
 			(remove_unused_layers no)
-			(net 2 "unconnected-(ACC1-AD0-Pad7)")
+			(net 22 "unconnected-(MPU1-AD0-Pad7)")
 			(pinfunction "AD0")
 			(pintype "bidirectional+no_connect")
@@
 			(layers "*.Cu" "*.Mask")
 			(remove_unused_layers no)
-			(net 4 "unconnected-(ACC1-INT-Pad8)")
+			(net 60 "unconnected-(MPU1-INT-Pad8)")
 			(pinfunction "INT")
 			(pintype "bidirectional+no_connect")
@@
 			)
 			(fill none)
-			(layer "Dwgs.User")
+			(layer "F.SilkS")
+		)
+		(fp_circle
+			(center -6 -22)
+			(end -5.5 -22)
+			(stroke
+				(width 0.1)
+				(type default)
+			)
+			(fill none)
+			(layer "F.SilkS")
 		)
 		(fp_rect
@@
 			(layer "F.SilkS")
 		)
+		(fp_rect
+			(start -2.54 -11.43)
+			(end 20.32 11.43)
+			(stroke
+				(width 0.1)
+				(type default)
+			)
+			(fill none)
+			(layer "F.SilkS")
+		)
 		(fp_line
 			(start 20.32 -11.43)
@@
 		(layer "F.Cu")
 		(at 142.24 108.712 90)
-		(property "Reference" "MPU1"
+		(property "Reference" "BME1"
 			(at -3.81 0 0)
 			(unlocked yes)
@@
 			)
 			(fill none)
-			(layer "Dwgs.User")
+			(layer "F.SilkS")
 		)
 		(fp_line
@@
 			(layers "*.Cu" "*.Mask")
 			(remove_unused_layers no)
-			(net 22 "Net-(IC1-A2)")
+			(net 2 "Net-(BME1-SCL)")
 			(pinfunction "SCL")
 			(pintype "input")
@@
 			(layers "*.Cu" "*.Mask")
 			(remove_unused_layers no)
-			(net 9 "Net-(IC1-A3)")
+			(net 4 "Net-(BME1-SDA)")
 			(pinfunction "SDA")
 			(pintype "bidirectional")
@@
 			(layers "*.Cu" "*.Mask")
 			(remove_unused_layers no)
-			(net 61 "unconnected-(MPU1-CSB-Pad5)")
+			(net 5 "unconnected-(BME1-CSB-Pad5)")
 			(pinfunction "CSB")
 			(pintype "input+no_connect")
@@
 			(layers "*.Cu" "*.Mask")
 			(remove_unused_layers no)
-			(net 60 "unconnected-(MPU1-SDO-Pad6)")
+			(net 1 "unconnected-(BME1-SDO-Pad6)")
 			(pinfunction "SDO")
 			(pintype "bidirectional+no_connect")
@@
 			(layers "*.Cu" "*.Mask")
 			(remove_unused_layers no)
-			(net 22 "Net-(IC1-A2)")
+			(net 2 "Net-(BME1-SCL)")
 			(pinfunction "A2")
 			(pintype "bidirectional")
@@
 			(layers "*.Cu" "*.Mask")
 			(remove_unused_layers no)
-			(net 9 "Net-(IC1-A3)")
+			(net 4 "Net-(BME1-SDA)")
 			(pinfunction "A3")
 			(pintype "bidirectional")
@@
 			(layers "*.Cu" "*.Mask")
 			(remove_unused_layers no)
-			(net 7 "Net-(ACC1-SDA)")
+			(net 7 "Net-(IC1-A4)")
 			(pinfunction "A4")
 			(pintype "bidirectional")
@@
 			(layers "*.Cu" "*.Mask")
 			(remove_unused_layers no)
-			(net 5 "Net-(ACC1-SCL)")
+			(net 8 "Net-(IC1-A5)")
 			(pinfunction "A5")
 			(pintype "bidirectional")
@@
 			)
 			(fill none)
-			(layer "B.Fab")
+			(layer "B.SilkS")
 		)
 		(fp_rect
@@
 			)
 			(fill none)
-			(layer "B.Fab")
+			(layer "B.SilkS")
 		)
 		(fp_text user "${REFERENCE}"
@@
 		(layer "F.SilkS")
 	)
-	(gr_rect
-		(start 133.5 100)
-		(end 151 111)
-		(stroke
-			(width 0.1)
-			(type default)
-		)
-		(fill none)
-		(layer "F.SilkS")
-	)
 	(gr_poly
 		(pts
@@
 		(layer "F.SilkS")
 	)
-	(gr_rect
-		(start 133.5 76.5)
-		(end 156 91.5)
-		(stroke
-			(width 0.1)
-			(type default)
-		)
-		(fill none)
-		(layer "F.SilkS")
-	)
 	(gr_poly
 		(pts
@@
 		(layer "F.SilkS")
 	)
-	(gr_rect
-		(start 151.5 92)
-		(end 174.5 115)
-		(stroke
-			(width 0.1)
-			(type default)
-		)
-		(fill none)
-		(layer "F.SilkS")
-	)
 	(gr_poly
 		(pts
@@
 		(layer "F.SilkS")
 	)
-	(gr_rect
-		(start 112 79.5)
-		(end 132 110)
-		(stroke
-			(width 0.1)
-			(type default)
-		)
-		(fill none)
-		(layer "F.SilkS")
-	)
 	(gr_poly
 		(pts
@@
 	)
 	(segment
+		(start 147.543 101.854)
+		(end 147.543 87.5215)
+		(width 0.254)
+		(layer "F.Cu")
+		(net 2)
+	)
+	(segment
+		(start 147.543 87.5215)
+		(end 148.7025 86.362)
+		(width 0.254)
+		(layer "F.Cu")
+		(net 2)
+	)
+	(segment
+		(start 140.97 108.712)
+		(end 147.543 102.139)
+		(width 0.254)
+		(layer "F.Cu")
+		(net 2)
+	)
+	(segment
+		(start 147.543 102.139)
+		(end 147.543 101.854)
+		(width 0.254)
+		(layer "F.Cu")
+		(net 2)
+	)
+	(segment
 		(start 156.718 84.582)
 		(end 153.67 81.534)
@@
 	)
 	(segment
-		(start 156.3225 86.362)
-		(end 148.9545 78.994)
+		(start 150.083 102.108)
+		(end 150.083 87.5215)
 		(width 0.254)
 		(layer "F.Cu")
-		(net 5)
+		(net 4)
 	)
 	(segment
-		(start 148.9545 78.994)
-		(end 148.59 78.994)
+		(start 150.083 102.139)
+		(end 150.083 102.108)
 		(width 0.254)
 		(layer "F.Cu")
-		(net 5)
+		(net 4)
 	)
 	(segment
-		(start 153.7825 86.362)
-		(end 146.4145 78.994)
+		(start 150.083 87.5215)
+		(end 151.2425 86.362)
 		(width 0.254)
 		(layer "F.Cu")
-		(net 7)
+		(net 4)
 	)
 	(segment
-		(start 146.4145 78.994)
-		(end 146.05 78.994)
+		(start 143.51 108.712)
+		(end 150.083 102.139)
 		(width 0.254)
 		(layer "F.Cu")
-		(net 7)
+		(net 4)
 	)
 	(segment
-		(start 150.083 102.108)
-		(end 150.083 87.5215)
+		(start 153.7825 86.362)
+		(end 146.4145 78.994)
 		(width 0.254)
 		(layer "F.Cu")
-		(net 9)
+		(net 7)
 	)
 	(segment
-		(start 150.083 102.139)
-		(end 150.083 102.108)
+		(start 146.4145 78.994)
+		(end 146.05 78.994)
 		(width 0.254)
 		(layer "F.Cu")
-		(net 9)
+		(net 7)
 	)
 	(segment
-		(start 150.083 87.5215)
-		(end 151.2425 86.362)
+		(start 156.3225 86.362)
+		(end 148.9545 78.994)
 		(width 0.254)
 		(layer "F.Cu")
-		(net 9)
+		(net 8)
 	)
 	(segment
-		(start 143.51 108.712)
-		(end 150.083 102.139)
+		(start 148.9545 78.994)
+		(end 148.59 78.994)
 		(width 0.254)
 		(layer "F.Cu")
-		(net 9)
+		(net 8)
 	)
 	(segment
@@
 	)
 	(segment
-		(start 147.543 101.854)
-		(end 147.543 87.5215)
-		(width 0.254)
-		(layer "F.Cu")
-		(net 22)
-	)
-	(segment
-		(start 147.543 87.5215)
-		(end 148.7025 86.362)
-		(width 0.254)
-		(layer "F.Cu")
-		(net 22)
-	)
-	(segment
-		(start 140.97 108.712)
-		(end 147.543 102.139)
-		(width 0.254)
-		(layer "F.Cu")
-		(net 22)
-	)
-	(segment
-		(start 147.543 102.139)
-		(end 147.543 101.854)
-		(width 0.254)
-		(layer "F.Cu")
-		(net 22)
-	)
-	(segment
