File: Panthera.kicad_sch (KiCad schematic)
At the start: 12 parts, among them IC1 TEENSY_4.1, SW1 SW_SPDT

Commit message: Updated PCB
Parts:
- renumbered MPU1 to BME1, ACC1 to MPU1
Changed lines of the file:
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@@
 		(dnp no)
 		(fields_autoplaced yes)
-		(property "Reference" "MPU1"
+		(property "Reference" "BME1"
 			(at 72.39 84.4549 0)
 			(effects
@@
 			(project ""
 				(path "/505f7bfa-4c2b-407e-860d-cc090cf0cd9e"
-					(reference "MPU1")
+					(reference "BME1")
 					(unit 1)
 				)
@@
 		(dnp no)
 		(fields_autoplaced yes)
-		(property "Reference" "ACC1"
-			(at 76.2 115.5701 0)
-			(effects
-				(font
-					(size 1.27 1.27)
-				)
-				(justify left)
+		(property "Reference" "MPU1"
+			(at 86.36 101.6 0)
+			(effects
+				(font
+					(size 1.27 1.27)
+				)
 			)
 		)
@@
 			(project ""
 				(path "/505f7bfa-4c2b-407e-860d-cc090cf0cd9e"
-					(reference "ACC1")
-					(unit 1)
-				)
+					(reference "MPU1")
+					(unit 1)
+				)
